File: kicad/LV Sensor - CAN/LV Sensor - CAN.kicad_pcb (KiCad board)
At the start: 2 copper layers, 26.2 x 30 mm, 9 parts, among them J2 Conn_01x09_Pin, U1 MCP2518FD-xJHA, U2 DSC1001DL5-020.0000T, U5 ATA6561-GAQW-N

Commit message: work faster 🍘
Parts:
- removed C4, C6: 100nF, Capacitor_SMD:C_1206_3216Metric_Pad1.33x1.80mm_HandSolder
- removed C5: 0.1uF, Capacitor_SMD:C_1206_3216Metric_Pad1.33x1.80mm_HandSolder
- removed C7: 0.01uF, Capacitor_SMD:C_1206_3216Metric_Pad1.33x1.80mm_HandSolder
- removed C8: 15pF, Capacitor_SMD:C_1206_3216Metric_Pad1.33x1.80mm_HandSolder
- removed J2: Conn_01x09_Pin, Connector_PinHeader_2.54mm:PinHeader_1x09_P2.54mm_Vertical
- removed U1: MCP2518FD-xJHA, LV-Sensor-Footprints-Lib:MCP2518FDT
- removed U2: DSC1001DL5-020.0000T, LV-Sensor-Footprints-Lib:CDFN4_2P5X2_MCH
- removed U5: ATA6561-GAQW-N, LV-Sensor-Footprints-Lib:SOIC8_4P9X3P9MC_MCH
Routing:
- net +5V: track 46.9 -> 0.00 mm
- net +3.3V: track 35.6 -> 0.00 mm
- net /CANL: track 13.4 -> 0.00 mm
- net /SDO: track 12.1 -> 0.00 mm
- net /CS: track 11.6 -> 0.00 mm
- net /SDIO: track 11.6 -> 0.00 mm
- net Net-(U1-OSC1): track 11.4 -> 0.00 mm
- net /SCK: track 11.1 -> 0.00 mm
- net /TXCAN: track 9.35 -> 0.00 mm
- net /RXCAN: track 4.44 -> 0.00 mm
- removed copper zone on B.Cu, net GND
- removed copper zone on F.Cu, net GND
Other:
- board outline removed
