File: kicad/LV Sensor - CAN/LV Sensor - CAN.kicad_pcb (KiCad board)
At the start: 2 copper layers, 29.8 x 29.2 mm, 9 parts, among them J2 Conn_01x09_Pin, U1 MCP2518FD-xJHA, U2 DSC1001DL5-020.0000T, U5 ATA6561-GAQW-N

Commit message: a
Parts:
- moved C7 13.5 mm to (114.4, 56.4), turned to -90 degrees
- moved U2 10.9 mm to (111.1, 56.6), turned to -90 degrees
- moved C4 8.02 mm to (115.6, 34.6), turned to 180 degrees
- moved C8 1.72 mm to (108.4, 49.8), turned to -90 degrees
Connections:
- J2 pad 3: +3.3V -> +5V
- J2 pad 9: +5V -> +3.3V
Routing:
- net +3.3V: track 84.2 -> 41.9 mm
- net +5V: track 4.64 -> 26.9 mm
- net /TXCAN: track 21.4 -> 10.9 mm
- net /*STANDBY: track 12.7 -> 11.8 mm

Commit message: 09-06-2025 Final CAN Board
Parts:
- moved U2 3.49 mm to (114.5, 55.8)
- moved C7 3.20 mm to (111.2, 56.4)
- moved C4 3.02 mm to (113.9, 37.1)
- moved U5 2.42 mm to (115.2, 41.1)
- moved C8 0.70 mm to (109.1, 49.8)
Connections:
- C7 pad 1: /*STANDBY -> Net-(U1-OSC1)
- C8 pad 2: /*STANDBY -> Net-(U1-OSC1)
- J2 pad 3: +5V -> +3.3V
- J2 pad 9: +3.3V -> +5V
- U1 pad 6: /*STANDBY -> Net-(U1-OSC1)
- U2 pad 1: /*STANDBY -> unconnected-(U2-*STANDBY-Pad1)
- U2 pad 3: unconnected-(U2-OUT-Pad3) -> Net-(U1-OSC1)
Routing:
- net +5V: track 26.9 -> 46.9 mm
- net /*STANDBY: track 11.8 -> 0.00 mm
- net Net-(U1-OSC1): track 0.00 -> 11.0 mm
- net /CANH: track 10.3 -> 0.00 mm
- net +3.3V: track 41.9 -> 35.6 mm
- net /CANL: track 9.80 -> 13.4 mm
- net /TXCAN: track 10.9 -> 7.65 mm
- net /RXCAN: track 6.85 -> 4.44 mm
Other:
- board size 29.8 x 29.2 mm -> 26.2 x 30 mm

Commit message: 09-05-2025 Final Again
Parts:
- moved C6 0.30 mm to (122.5, 42.0)
Connections:
- U1 pad 7: unconnected-(U1-VSS-Pad7) -> GND
Routing:
- net /TXCAN: track 7.65 -> 9.35 mm
Changed lines of the file:
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@@
 	(net 14 "/CANL")
 	(net 15 "/CANH")
-	(net 16 "unconnected-(U1-VSS-Pad7)")
-	(net 17 "unconnected-(U2-*STANDBY-Pad1)")
+	(net 16 "unconnected-(U2-*STANDBY-Pad1)")
 	(footprint "LV-Sensor-Footprints-Lib:MCP2518FDT"
 		(layer "F.Cu")
@@
 			(net 6 "unconnected-(U1-~{INT}-Pad4)")
 			(pinfunction "~{INT}")
-			(pintype "output")
+			(pintype "output+no_connect")
 		)
 		(pad "5" smd roundrect
@@
 			(layers "F.Cu" "F.Mask" "F.Paste")
 			(roundrect_rratio 0.25)
-			(net 16 "unconnected-(U1-VSS-Pad7)")
+			(net 1 "GND")
 			(pinfunction "VSS")
 			(pintype "power_in")
@@
 			(net 10 "unconnected-(U1-~{INT1}{slash}GPIO1-Pad8)")
 			(pinfunction "~{INT1}/GPIO1")
-			(pintype "bidirectional")
+			(pintype "bidirectional+no_connect")
 		)
 		(pad "9" smd roundrect
@@
 			(net 13 "unconnected-(U1-~{INT0}{slash}GPIO0{slash}XSTBY-Pad9)")
 			(pinfunction "~{INT0}/GPIO0/XSTBY")
-			(pintype "bidirectional")
+			(pintype "bidirectional+no_connect")
 		)
 		(pad "10" smd roundrect
@@
 			(size 0.9548 0.5992)
 			(layers "F.Cu" "F.Mask" "F.Paste")
-			(net 17 "unconnected-(U2-*STANDBY-Pad1)")
+			(net 16 "unconnected-(U2-*STANDBY-Pad1)")
 			(pinfunction "*STANDBY")
 			(pintype "input+no_connect")
@@
 	(footprint "Capacitor_SMD:C_1206_3216Metric_Pad1.33x1.80mm_HandSolder"
 		(layer "F.Cu")
-		(at 122.2 42 -90)
+		(at 122.5 42 -90)
 		(descr "Capacitor SMD 1206 (3216 Metric), square (rectangular) end terminal, IPC-7351 nominal with elongated pad for handsoldering. (Body size source: IPC-SM-782 page 76, https://www.pcb-3d.com/wordpress/wp-content/uploads/ipc-sm-782a_amendment_1_and_2.pdf), generated with kicad-footprint-generator")
 		(tags "capacitor handsolder")
@@
 	)
 	(segment
-		(start 110.499 54.1365)
-		(end 110.499 52.102636)
+		(start 111.2 54.8375)
+		(end 110 53.6375)
 		(width 0.5)
 		(layer "F.Cu")
@@
 	)
 	(segment
-		(start 111.241636 51.36)
-		(end 112.025 51.36)
-		(width 0.5)
-		(layer "F.Cu")
-		(net 4)
-	)
-	(segment
 		(start 109.1025 51.36)
 		(end 109.1 51.3625)
@@
 	)
 	(segment
-		(start 110.499 52.102636)
+		(start 110 52.601636)
 		(end 111.241636 51.36)
 		(width 0.5)
@@
 	)
 	(segment
-		(start 111.2 54.8375)
-		(end 110.499 54.1365)
+		(start 110 53.6375)
+		(end 110 52.601636)
+		(width 0.5)
+		(layer "F.Cu")
+		(net 4)
+	)
+	(segment
+		(start 111.241636 51.36)
+		(end 112.025 51.36)
 		(width 0.5)
 		(layer "F.Cu")
@@
 	)
 	(segment
-		(start 113.7362 39.195)
-		(end 112.2342 39.195)
+		(start 110.4 40)
+		(end 110.4 43.385)
 		(width 0.5)
 		(layer "F.Cu")
@@
 	)
 	(segment
-		(start 111.725001 44.710001)
-		(end 112.025 45.01)
+		(start 113.7362 39.195)
+		(end 111.205 39.195)
 		(width 0.5)
 		(layer "F.Cu")
@@
 	)
 	(segment
-		(start 111.725001 39.704199)
-		(end 111.725001 44.710001)
+		(start 111.205 39.195)
+		(end 110.4 40)
 		(width 0.5)
 		(layer "F.Cu")
@@
 	)
 	(segment
-		(start 112.2342 39.195)
-		(end 111.725001 39.704199)
+		(start 110.4 43.385)
+		(end 112.025 45.01)
 		(width 0.5)
 		(layer "F.Cu")
@@
 		(filled_areas_thickness no)
 		(fill yes
-			(thermal_gap 0.5)
+			(thermal_gap 0)
 			(thermal_bridge_width 0.5)
+			(island_removal_mode 1)
+			(island_area_min 10)
 		)
 		(polygon
@@
 		(filled_areas_thickness no)
 		(fill yes
-			(thermal_gap 0.5)
+			(thermal_gap 0)
 			(thermal_bridge_width 0.5)
 		)

Commit message: 09-10-25
Parts:
- removed C5: 0.1uF, Capacitor_SMD:C_1206_3216Metric_Pad1.33x1.80mm_HandSolder
- removed C7: 0.01uF, Capacitor_SMD:C_1206_3216Metric_Pad1.33x1.80mm_HandSolder
- added C1: 100nF, Capacitor_SMD:C_1206_3216Metric_Pad1.33x1.80mm_HandSolder, F.Cu at (122.6, 36.2)
- added C2: 100nF, Capacitor_SMD:C_1206_3216Metric_Pad1.33x1.80mm_HandSolder, F.Cu at (125.4, 36.4)
- added TP1: TestPoint, Connector_Pin:Pin_D1.0mm_L10.0mm, F.Cu at (120.7, 55.9)
- added TP2: TestPoint, Connector_Pin:Pin_D1.0mm_L10.0mm, F.Cu at (123.7, 52.8)
- added TP3: TestPoint, Connector_Pin:Pin_D1.0mm_L10.0mm, F.Cu at (109.1, 46.3)
- added TP4: TestPoint, Connector_Pin:Pin_D1.0mm_L10.0mm, F.Cu at (111.6, 49.4)
- added TP5: TestPoint, Connector_Pin:Pin_D1.0mm_L10.0mm, F.Cu at (108.8, 51.7)
- added TP6: TestPoint, Connector_Pin:Pin_D1.0mm_L10.0mm, F.Cu at (116.6, 36.7)
- moved C6 11.8 mm to (112.5, 35.6), turned to 135 degrees
- moved C8 7.69 mm to (109.4, 57.5), turned to -45 degrees
- moved C4 6.57 mm to (119.3, 33.4), turned to 45 degrees
- moved U2 3.01 mm to (111.6, 55.0), turned to 135 degrees
- moved U1 2.96 mm to (117.5, 49.4)
- moved U5 2.15 mm to (113.0, 41.1)
- moved J2 1.40 mm to (128.6, 35.4)
Connections:
- net /RXCAN renamed Net-(U1-RXCAN)
- net /TXCAN renamed Net-(U1-TXCAN)
- C4 pad 1: +5V -> +3.3V
- C8 pad 1: GND -> +3V3
- C8 pad 2: Net-(U1-OSC1) -> GND
- J2 pad 1: /CANH -> GND
- J2 pad 2: /CANL -> +5V
- J2 pad 4: GND -> Net-(J2-Pin_4)
- J2 pad 5: /CS -> Net-(J2-Pin_5)
- J2 pad 6: /SDO -> Net-(J2-Pin_6)
- J2 pad 7: /SDIO -> Net-(J2-Pin_7)
- J2 pad 8: /SCK -> /CAN_H
- J2 pad 9: +5V -> /CAN_L
- U1 pad 10: /SCK -> Net-(J2-Pin_7)
- U1 pad 11: /SDIO -> Net-(J2-Pin_6)
- U1 pad 12: /SDO -> Net-(J2-Pin_5)
- U1 pad 13: /CS -> Net-(J2-Pin_4)
- U1 pad 3: GND -> Net-(U1-CLKO/SOF)
- U1 pad 4: unconnected-(U1-~{INT}-Pad4) -> Net-(U1-~{INT})
- U1 pad 5: GND -> Net-(U1-OSC2)
- U1 pad 8: unconnected-(U1-~{INT1}/GPIO1-Pad8) -> Net-(U1-~{INT1}/GPIO1)
- U1 pad 9: unconnected-(U1-~{INT0}/GPIO0/XSTBY-Pad9) -> Net-(U1-~{INT0}/GPIO0/XSTBY)
- U2 pad 4: +3.3V -> +3V3
- U5 pad 6: /CANL -> /CAN_L
- U5 pad 7: /CANH -> /CAN_H
- U5 pad 8: GND -> Net-(U5-STBY)
Routing:
- net /CAN_H: track 0.00 -> 31.0 mm
- net /CAN_L: track 0.00 -> 31.0 mm
- net +5V: track 46.9 -> 31.8 mm
- net /CANL: track 13.4 -> 0.00 mm
- net /SDO: track 12.1 -> 0.00 mm
- net /CS: track 11.6 -> 0.00 mm
- net /SDIO: track 11.6 -> 0.00 mm
- net /SCK: track 11.1 -> 0.00 mm
- net Net-(J2-Pin_4): track 0.00 -> 9.86 mm
- net Net-(J2-Pin_5): track 0.00 -> 9.33 mm
- net Net-(J2-Pin_6): track 0.00 -> 8.81 mm
- net Net-(J2-Pin_7): track 0.00 -> 8.31 mm
- net Net-(U1-OSC1): track 11.4 -> 4.10 mm
- net Net-(U1-CLKO/SOF): track 0.00 -> 6.62 mm
- net Net-(U1-OSC2): track 0.00 -> 6.01 mm
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Other:
- board size 26.2 x 30 mm -> 26.8 x 33.5 mm

Commit message: ljklj
Changed notation 3V3 to 3.3V

Co-Authored-By: Manish Shrestha <manish.shr006@gmail.com>
Connections:
- C8 pad 1: +3V3 -> +3.3V
- U2 pad 4: +3V3 -> +3.3V
Routing:
- net +3.3V: track 34.7 -> 37.4 mm
- net +3V3: track 2.71 -> 0.00 mm
