File: kicad/LV Sensor - CAN/LV Sensor - CAN.kicad_sch (KiCad schematic)
At the start: 4 parts, among them U1 ATA00F18S-L, U2 MCP251863T-H-SS, U3 DSC1001DL5-020.0000T

Commit message: 09-05-2025 "Finished" LV-Sensor-Can Board
Parts:
- removed C1: C, symbol Device:C
- removed U1: ATA00F18S-L, LV-Sensor-Footprints-Lib:SOIC8_4P9X3P9MC_MCH, symbol LV-Sensor-Lib:ATA6561-GAQW-N
- removed U2: MCP251863T-H-SS, LV-Sensor-Footprints-Lib:MCP2518FDT, symbol LV-Sensor-Lib:MCP2517FD-xJHA
- removed U3: DSC1001DL5-020.0000T, LV-Sensor-Footprints-Lib:CDFN4_2P5X2_MCH, symbol LV-Sensor-Lib:DSC1001DL5-020.0000T
- added C4, C6: 100nF, Capacitor_SMD:C_1206_3216Metric_Pad1.33x1.80mm_HandSolder, symbol Device:C
- added C5: 0.1uF, Capacitor_SMD:C_1206_3216Metric_Pad1.33x1.80mm_HandSolder, symbol Device:C
- added C7: 0.01uF, Capacitor_SMD:C_1206_3216Metric_Pad1.33x1.80mm_HandSolder, symbol Device:C_Small
- added C8: 15pF, Capacitor_SMD:C_1206_3216Metric_Pad1.33x1.80mm_HandSolder, symbol Device:C_Small
- added J2: Conn_01x09_Pin, Connector_PinHeader_2.54mm:PinHeader_1x09_P2.54mm_Vertical, symbol Connector:Conn_01x09_Pin
- added U1: MCP2518FD-xJHA, LV-Sensor-Footprints-Lib:MCP2518FDT, symbol LV-Sensor-Lib:MCP2517FD-xJHA
- added U2: DSC1001DL5-020.0000T, LV-Sensor-Footprints-Lib:CDFN4_2P5X2_MCH, symbol LV-Sensor-Lib:DSC1001DL5-020.0000T
- added U5: ATA6561-GAQW-N, LV-Sensor-Footprints-Lib:SOIC8_4P9X3P9MC_MCH, symbol LV-Sensor-Lib:ATA6561-GAQW-N
Connections:
- net GND: now also C4.2, C5.1, C6.2, C8.1, J2.4 (Pin_4), U1.3 (CLKO/SOF), U1.5 (OSC2), U2.2 (GND), U5.2 (GND), U5.8 (STBY)
- new net *STANDBY: C7.1, C8.2, U1.6 (OSC1), U2.1 (*STANDBY)
- new net +3.3V: C5.2, C6.1, C7.2, J2.3 (Pin_3), U1.14 (VDD), U2.4 (VDD), U5.5 (VIO)
- new net +5V: C4.1, J2.9 (Pin_9), U5.3 (VCC)
- new net CANH: J2.1 (Pin_1), U5.7 (CANH)
- new net CANL: J2.2 (Pin_2), U5.6 (CANL)
- new net CS: J2.5 (Pin_5), U1.13 (~{CS})
- new net RXCAN: U1.2 (RXCAN), U5.4 (RXD)
- new net SCK: J2.8 (Pin_8), U1.10 (SCK)
- new net SDIO: J2.7 (Pin_7), U1.11 (SDI)
- new net SDO: J2.6 (Pin_6), U1.12 (SDO)
- new net TXCAN: U1.1 (TXCAN), U5.1 (TXD)
- no-connect marks 0 -> 1
Other:
- note added: "CAN Stand-alone Controller"

Commit message: everything is nasty
Connections:
- net +3.3V: now also J2.9 (Pin_9); no longer J2.3 (Pin_3)
- net +5V: now also J2.3 (Pin_3); no longer J2.9 (Pin_9)
Changed lines of the file:
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@@
 	(symbol
 		(lib_id "power:+5V")
-		(at 88.9 101.6 270)
+		(at 88.9 86.36 270)
 		(unit 1)
 		(exclude_from_sim no)
@@
 		(fields_autoplaced yes)
 		(property "Reference" "#PWR02"
-			(at 85.09 101.6 0)
+			(at 85.09 86.36 0)
 			(effects
 				(font
@@
 		)
 		(property "Value" "+5V"
-			(at 92.71 101.5999 90)
+			(at 92.71 86.3599 90)
 			(effects
 				(font
@@
 		)
 		(property "Footprint" ""
-			(at 88.9 101.6 0)
+			(at 88.9 86.36 0)
 			(effects
 				(font
@@
 		)
 		(property "Datasheet" ""
-			(at 88.9 101.6 0)
+			(at 88.9 86.36 0)
 			(effects
 				(font
@@
 		)
 		(property "Description" "Power symbol creates a global label with name \"+5V\""
-			(at 88.9 101.6 0)
+			(at 88.9 86.36 0)
 			(effects
 				(font
@@
 	(symbol
 		(lib_id "power:+3.3V")
-		(at 88.9 86.36 270)
+		(at 88.9 101.6 270)
 		(unit 1)
 		(exclude_from_sim no)
@@
 		(dnp no)
 		(property "Reference" "#PWR03"
-			(at 85.09 86.36 0)
+			(at 85.09 101.6 0)
 			(effects
 				(font
@@
 		)
 		(property "Value" "+3.3V"
-			(at 93.218 86.36 90)
+			(at 93.218 101.6 90)
 			(effects
 				(font
@@
 		)
 		(property "Footprint" ""
-			(at 88.9 86.36 0)
+			(at 88.9 101.6 0)
 			(effects
 				(font
@@
 		)
 		(property "Datasheet" ""
-			(at 88.9 86.36 0)
+			(at 88.9 101.6 0)
 			(effects
 				(font
@@
 		)
 		(property "Description" "Power symbol creates a global label with name \"+3.3V\""
-			(at 88.9 86.36 0)
-			(effects
-				(font
+			(at 88.9 101.6 0)
+			(effects
+				(font

Commit message: 09-06-2025 Final CAN Board
Connections:
- net +3.3V: now also J2.3 (Pin_3); no longer J2.9 (Pin_9)
- net +5V: now also J2.9 (Pin_9); no longer J2.3 (Pin_3)
- net at U2.3 (OUT): now also C7.1, C8.2, U1.6 (OSC1)
- removed net *STANDBY: C7.1, C8.2, U1.6 (OSC1), U2.1 (*STANDBY)
Changed lines of the file:
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@@
+	)
+	(junction
+		(at 125.73 120.65)
+		(diameter 0)
+		(color 0 0 0 0)
+	)
+	(junction
+		(at 220.98 113.03)
+		(diameter 0)
+		(color 0 0 0 0)
+	)
+	(junction
+		(at 171.45 113.03)
+		(diameter 0)
+		(color 0 0 0 0)
+	)
+	(junction
+		(at 116.84 120.65)
+		(diameter 0)
+		(color 0 0 0 0)
+	)
+	(junction
+		(at 118.11 91.44)
+		(diameter 0)
+		(color 0 0 0 0)
+	)
+	(junction
+		(at 116.84 114.3)
+		(diameter 0)
+		(color 0 0 0 0)
 	)
 	(junction
@@
 		(color 0 0 0 0)
 	)
-	(junction
-		(at 125.73 120.65)
-		(diameter 0)
-		(color 0 0 0 0)
-	)
-	(junction
-		(at 220.98 113.03)
-		(diameter 0)
-		(color 0 0 0 0)
-	)
-	(junction
-		(at 171.45 113.03)
-		(diameter 0)
-		(color 0 0 0 0)
-	)
-	(junction
-		(at 118.11 91.44)
-		(diameter 0)
-		(color 0 0 0 0)
-	)
-	(junction
-		(at 116.84 114.3)
-		(diameter 0)
-		(color 0 0 0 0)
-	)
-	(junction
-		(at 116.84 120.65)
-		(diameter 0)
-		(color 0 0 0 0)
-	)
 	(no_connect
-		(at 113.03 118.11)
+		(at 82.55 114.3)
 	)
 	(wire
@@
 	(wire
 		(pts
+			(xy 125.73 111.76) (xy 129.54 111.76)
+		)
+		(stroke
+			(width 0)
+			(type default)
+		)
+	)
+	(wire
+		(pts
+			(xy 125.73 111.76) (xy 125.73 114.3)
+		)
+		(stroke
+			(width 0)
+			(type default)
+		)
+	)
+	(wire
+		(pts
+			(xy 121.92 106.68) (xy 121.92 111.76)
+		)
+		(stroke
+			(width 0)
+			(type default)
+		)
+	)
+	(wire
+		(pts
+			(xy 113.03 120.65) (xy 113.03 118.11)
+		)
+		(stroke
+			(width 0)
+			(type default)
+		)
+	)
+	(wire
+		(pts
+			(xy 88.9 86.36) (xy 85.09 86.36)
+		)
+		(stroke
+			(width 0)
+			(type default)
+		)
+	)
+	(wire
+		(pts
+			(xy 128.27 114.3) (xy 128.27 120.65)
+		)
+		(stroke
+			(width 0)
+			(type default)
+		)
+	)
+	(wire
+		(pts
+			(xy 88.9 81.28) (xy 85.09 81.28)
+		)
+		(stroke
+			(width 0)
+			(type default)
+		)
+	)
+	(wire
+		(pts
 			(xy 69.85 118.11) (xy 82.55 118.11)
 		)
@@
 	(wire
 		(pts
-			(xy 125.73 111.76) (xy 129.54 111.76)
-		)
-		(stroke
-			(width 0)
-			(type default)
-		)
-	)
-	(wire
-		(pts
-			(xy 125.73 111.76) (xy 125.73 114.3)
-		)
-		(stroke
-			(width 0)
-			(type default)
-		)
-	)
-	(wire
-		(pts
-			(xy 121.92 106.68) (xy 121.92 111.76)
-		)
-		(stroke
-			(width 0)
-			(type default)
-		)
-	)
-	(wire
-		(pts
-			(xy 128.27 114.3) (xy 128.27 120.65)
-		)
-		(stroke
-			(width 0)
-			(type default)
-		)
-	)
-	(wire
-		(pts
-			(xy 88.9 81.28) (xy 85.09 81.28)
-		)
-		(stroke
-			(width 0)
-			(type default)
-		)
-	)
-	(wire
-		(pts
 			(xy 212.09 113.03) (xy 220.98 113.03)
 		)
@@
 	(wire
 		(pts
-			(xy 113.03 123.19) (xy 116.84 123.19)
-		)
-		(stroke
-			(width 0)
-			(type default)
-		)
-	)
-	(wire
-		(pts
 			(xy 116.84 119.38) (xy 116.84 120.65)
 		)
@@
 	(wire
 		(pts
+			(xy 88.9 101.6) (xy 85.09 101.6)
+		)
+		(stroke
+			(width 0)
+			(type default)
+		)
+	)
+	(wire
+		(pts
 			(xy 69.85 106.68) (xy 121.92 106.68)
 		)
@@
 	(wire
 		(pts
-			(xy 116.84 123.19) (xy 116.84 120.65)
+			(xy 116.84 120.65) (xy 113.03 120.65)
 		)
 		(stroke
@@
 	(wire
 		(pts
-			(xy 88.9 86.36) (xy 85.09 86.36)
-		)
-		(stroke
-			(width 0)
-			(type default)
-		)
-	)
-	(wire
-		(pts
 			(xy 167.64 113.03) (xy 171.45 113.03)
 		)
@@
 		(pts
 			(xy 113.03 114.3) (xy 116.84 114.3)
-		)
-		(stroke
-			(width 0)
-			(type default)
-		)
-	)
-	(wire
-		(pts
-			(xy 88.9 101.6) (xy 85.09 101.6)
 		)
 		(stroke
@@
 		)
 	)
-	(hierarchical_label "*STANDBY"
-		(shape input)
-		(at 82.55 114.3 180)
-		(effects
-			(font
-				(size 1.27 1.27)
-			)
-			(justify right)
-		)
-	)
 	(hierarchical_label "RXCAN"
 		(shape input)
@@
 			)
 			(justify left)
-		)
-	)
-	(hierarchical_label "*STANDBY"
-		(shape input)
-		(at 113.03 123.19 180)
-		(effects
-			(font
-				(size 1.27 1.27)
-			)
-			(justify right)
 		)
 	)
@@
 	(symbol
 		(lib_id "power:+5V")
-		(at 88.9 86.36 270)
+		(at 88.9 101.6 270)
 		(unit 1)
 		(exclude_from_sim no)
@@
 		(fields_autoplaced yes)
 		(property "Reference" "#PWR02"
-			(at 85.09 86.36 0)
+			(at 85.09 101.6 0)
 			(effects
 				(font
@@
 		)
 		(property "Value" "+5V"
-			(at 92.71 86.3599 90)
+			(at 92.71 101.5999 90)
 			(effects
 				(font
@@
 		)
 		(property "Footprint" ""
-			(at 88.9 86.36 0)
+			(at 88.9 101.6 0)
 			(effects
 				(font
@@
 		)
 		(property "Datasheet" ""
-			(at 88.9 86.36 0)
+			(at 88.9 101.6 0)
 			(effects
 				(font
@@
 		)
 		(property "Description" "Power symbol creates a global label with name \"+5V\""
-			(at 88.9 86.36 0)
+			(at 88.9 101.6 0)
 			(effects
 				(font
@@
 	(symbol
 		(lib_id "power:+3.3V")
-		(at 88.9 101.6 270)
+		(at 88.9 86.36 270)
 		(unit 1)
 		(exclude_from_sim no)
@@
 		(dnp no)
 		(property "Reference" "#PWR03"
-			(at 85.09 101.6 0)
+			(at 85.09 86.36 0)
 			(effects
 				(font
@@
 		)
 		(property "Value" "+3.3V"
-			(at 93.218 101.6 90)
+			(at 93.218 86.36 90)
 			(effects
 				(font
@@
 		)
 		(property "Footprint" ""
-			(at 88.9 101.6 0)
+			(at 88.9 86.36 0)
 			(effects
 				(font
@@
 		)
 		(property "Datasheet" ""
-			(at 88.9 101.6 0)
+			(at 88.9 86.36 0)
 			(effects
 				(font
@@
 		)
 		(property "Description" "Power symbol creates a global label with name \"+3.3V\""
-			(at 88.9 101.6 0)
-			(effects
-				(font
+			(at 88.9 86.36 0)
+			(effects
+				(font

Commit message: 09-06-2025 Fixed Some Changes
Connections:
- net GND: now also U1.7 (VSS)
Changed lines of the file:
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@@
+	)
+	(junction
+		(at 129.54 121.92)
+		(diameter 0)
+		(color 0 0 0 0)
 	)
 	(junction
@@
 	(wire
 		(pts
+			(xy 129.54 121.92) (xy 129.54 123.19)
+		)
+		(stroke
+			(width 0)
+			(type default)
+		)
+	)
+	(wire
+		(pts
 			(xy 125.73 111.76) (xy 125.73 114.3)
 		)
@@
 	(wire
 		(pts
+			(xy 129.54 116.84) (xy 129.54 121.92)
+		)
+		(stroke
+			(width 0)
+			(type default)
+		)
+	)
+	(wire
+		(pts
 			(xy 116.84 119.38) (xy 116.84 120.65)
 		)
@@
 		(pts
 			(xy 220.98 113.03) (xy 220.98 120.65)
+		)
+		(stroke
+			(width 0)
+			(type default)
+		)
+	)
+	(wire
+		(pts
+			(xy 129.54 121.92) (xy 132.08 121.92)
 		)
 		(stroke
@@
 		)
 	)
+	(hierarchical_label "VSS"
+		(shape input)
+		(at 129.54 104.14 180)
+		(effects
+			(font
+				(size 1.27 1.27)
+			)
+			(justify right)
+		)
+	)
 	(hierarchical_label "TXCAN"
 		(shape input)
@@
 		(shape input)
 		(at 220.98 104.14 0)
+		(effects
+			(font
+				(size 1.27 1.27)
+			)
+			(justify left)
+		)
+	)
+	(hierarchical_label "VSS"
+		(shape input)
+		(at 132.08 121.92 0)
 		(effects
 			(font
@@
 	(symbol
 		(lib_id "power:GND")
-		(at 129.54 104.14 270)
+		(at 129.54 123.19 0)
 		(unit 1)
 		(exclude_from_sim no)
@@
 		(fields_autoplaced yes)
 		(property "Reference" "#PWR015"
-			(at 123.19 104.14 0)
+			(at 129.54 129.54 0)
 			(effects
 				(font
@@
 		)
 		(property "Value" "GND"
-			(at 125.73 104.1399 90)
-			(effects
-				(font
-					(size 1.27 1.27)
-				)
-				(justify right)
+			(at 129.54 128.27 0)
+			(effects
+				(font
+					(size 1.27 1.27)
+				)
 			)
 		)
 		(property "Footprint" ""
-			(at 129.54 104.14 0)
+			(at 129.54 123.19 0)
 			(effects
 				(font
@@
 		)
 		(property "Datasheet" ""
-			(at 129.54 104.14 0)
+			(at 129.54 123.19 0)
 			(effects
 				(font
@@
 		)
 		(property "Description" "Power symbol creates a global label with name \"GND\" , ground"
-			(at 129.54 104.14 0)
-			(effects
-				(font
+			(at 129.54 123.19 0)
+			(effects
+				(font

Commit message: 09-05-2025 Final Again
Connections:
- no-connect marks 1 -> 4
Other:
- moved on the sheet: C4, C6, U5

Commit message: work faster 🍘
Parts:
- removed C4, C6: 100nF, Capacitor_SMD:C_1206_3216Metric_Pad1.33x1.80mm_HandSolder, symbol Device:C
- removed C5: 0.1uF, Capacitor_SMD:C_1206_3216Metric_Pad1.33x1.80mm_HandSolder, symbol Device:C
- removed C7: 0.01uF, Capacitor_SMD:C_1206_3216Metric_Pad1.33x1.80mm_HandSolder, symbol Device:C_Small
- removed C8: 15pF, Capacitor_SMD:C_1206_3216Metric_Pad1.33x1.80mm_HandSolder, symbol Device:C_Small
- removed J2: Conn_01x09_Pin, Connector_PinHeader_2.54mm:PinHeader_1x09_P2.54mm_Vertical, symbol Connector:Conn_01x09_Pin
- removed U1: MCP2518FD-xJHA, LV-Sensor-Footprints-Lib:MCP2518FDT, symbol LV-Sensor-Lib:MCP2517FD-xJHA
- removed U2: DSC1001DL5-020.0000T, LV-Sensor-Footprints-Lib:CDFN4_2P5X2_MCH, symbol LV-Sensor-Lib:DSC1001DL5-020.0000T
- removed U5: ATA6561-GAQW-N, LV-Sensor-Footprints-Lib:SOIC8_4P9X3P9MC_MCH, symbol LV-Sensor-Lib:ATA6561-GAQW-N
- added C1, C10, C2, C9: 100nF, Capacitor_SMD:C_1206_3216Metric_Pad1.33x1.80mm_HandSolder, symbol Device:C
- added C3: 15pF, Capacitor_SMD:C_1206_3216Metric_Pad1.33x1.80mm_HandSolder, symbol Device:C_Small
- added J1: Conn_01x09_Pin, Connector_PinHeader_2.54mm:PinHeader_1x09_P2.54mm_Vertical, symbol Connector:Conn_01x09_Pin
- added TP1, TP2, TP3, TP4, TP5, TP6: TestPoint, Connector_Pin:Pin_D1.0mm_L10.0mm, symbol Connector:TestPoint
- added U3: DSC1001DL5-020.0000T, LV-Sensor-Footprints-Lib:CDFN4_2P5X2_MCH, symbol LV-Sensor-Lib:DSC1001DL5-020.0000T
- added U4: MCP2518FD-xJHA, LV-Sensor-Footprints-Lib:MCP2518FDT, symbol LV-Sensor-Lib:MCP2517FD-xJHA
- added U6: ATA6561-GAQW-N, LV-Sensor-Footprints-Lib:SOIC8_4P9X3P9MC_MCH, symbol LV-Sensor-Lib:ATA6561-GAQW-N
Connections:
- net +3.3V: now also C2.1, C3.1, C9.1, J1.2 (Pin_2), U3.4 (VDD), U4.14 (VDD), U6.5 (VIO)
- net +5V: now also C1.1, C10.1, J1.3 (Pin_3), U6.3 (VCC)
- net CS: now also J1.4 (Pin_4), U4.13 (~{CS})
- net GND: now also C1.2, C10.2, C2.2, C3.2, C9.2, J1.1 (Pin_1), U3.2 (GND), U4.7 (VSS), U6.2 (GND)
- net SCK: now also J1.7 (Pin_7), U4.10 (SCK)
- net SDO: now also J1.5 (Pin_5), U4.12 (SDO)
- new net: U3.3 (OUT), U4.6 (OSC1)
- new net: U4.1 (TXCAN), U6.1 (TXD)
- new net: U4.2 (RXCAN), U6.4 (RXD)
- new net: TP3.1, U4.3 (CLKO/SOF)
- new net: TP4.1, U4.4 (~{INT})
- new net: TP5.1, U4.5 (OSC2)
- new net: TP1.1, U4.8 (~{INT1}/GPIO1)
- new net: TP2.1, U4.9 (~{INT0}/GPIO0/XSTBY)
- new net: TP6.1, U6.8 (STBY)
- new net CAN_H: J1.8 (Pin_8), U6.7 (CANH)
- new net CAN_L: J1.9 (Pin_9), U6.6 (CANL)
- new net SDI: J1.6 (Pin_6), U4.11 (SDI)
- no-connect marks 4 -> 1
Other:
- note added: "pg.4 : leave floating?"
- note added: "size unspecified"
- note removed: "CAN Stand-alone Controller"
