File: kicad/LV Sensor.kicad_sch (KiCad schematic)
At the start: 71 parts, among them J16 USB_B_Micro, U1 AP63205WU-7, U10 LM2662MX/NOPB, U2 XMSM0C1104SPW20R, U3 FT231XS-R, U4 AP63203WU-7, U5 TLV77325PDBVR, U6 MCP2518FD-xJHA, U7 DSC1001DL5-020.0000T, U8 ADS114S06BIPBSR, U9 ATA6561-GAQW-N

Commit message: 5y5y
45y45

Co-Authored-By: Manish Shrestha <manish.shr006@gmail.com>
Parts:
- removed C19: 15pF, Capacitor_SMD:C_1206_3216Metric_Pad1.33x1.80mm_HandSolder, symbol Device:C_Small
- removed C2: 100n, Capacitor_SMD:C_1206_3216Metric_Pad1.33x1.80mm_HandSolder, symbol Device:C_Small
- added SW1: SW_Push, symbol Switch:SW_Push
Connections:
- net +2V5: now also C17.2, C21.2, U8.26 (AVDD); no longer C21.1, U8.27 (AVSS), U8.28 (AVSS-SW)
- net -2V5: now also C21.1, U8.27 (AVSS), U8.28 (AVSS-SW); no longer C17.2, C21.2, U8.26 (AVDD)
- net GND: now also SW1.2
- net PA1: now also U8.9 (CS_N)
- net at U2.8 (PA2), U6.13 (~{CS}): no longer U8.9 (CS_N)
- net at R1.1, U2.4 (NRST): now also SW1.1
- no-connect marks 31 -> 30
Other:
- note removed: "size unspecified"
- moved on the sheet: C18

Commit message: aerg
Completely fixed everything

Co-Authored-By: Manish Shrestha <manish.shr006@gmail.com>
Parts:
- removed C17: 1uF, Capacitor_SMD:C_1206_3216Metric_Pad1.33x1.80mm_HandSolder, symbol Device:C_Small
- removed C18: 0.1uF, Capacitor_SMD:C_1206_3216Metric_Pad1.33x1.80mm_HandSolder, symbol Device:C_Small
- removed C21: 330nF, Capacitor_SMD:C_1206_3216Metric_Pad1.33x1.80mm_HandSolder, symbol Device:C_Small
- removed C22, C27: 47uF, Capacitor_SMD:C_1206_3216Metric_Pad1.33x1.80mm_HandSolder, symbol Device:C_Small
- removed C23, C24, C25, C26: 100nF, Capacitor_SMD:C_1206_3216Metric_Pad1.33x1.80mm_HandSolder, symbol Device:C
- removed D1, D2, D3, D4, D5, D6, D7, D8: 5.1V, symbol Device:D_Zener_Small
- removed R10, R14, R18, R5: 32k, symbol Device:R_Small_US
- removed R11, R15, R19, R4: 24k, symbol Device:R_Small_US
- removed R12, R16, R7, R8: 400, symbol Device:R_Small_US
- removed R13, R17, R6, R9: 600, symbol Device:R_Small_US
- removed TP3, TP4, TP5, TP6, TP7, TP8: TestPoint, symbol Connector:TestPoint
- removed U10: LM2662MX/NOPB, LV-Sensor-Footprints-Lib:M08A, symbol LV-Sensor-Lib:LM2662MX_NOPB
- removed U6: MCP2518FD-xJHA, LV-Sensor-Footprints-Lib:MCP2518FDT, symbol LV-Sensor-Lib:MCP2517FD-xJHA
- removed U7: DSC1001DL5-020.0000T, LV-Sensor-Footprints-Lib:CDFN4_2P5X2_MCH, symbol LV-Sensor-Lib:DSC1001DL5-020.0000T
- removed U8: ADS114S06BIPBSR, LV-Sensor-Footprints-Lib:PBS0032A_N, symbol LV-Sensor-Lib:ADS114S06BIPBSR
- added C1, C2, C7: 0.1µF, symbol Device:C
- added C17: 330nF, symbol Device:C
- added C18: 47µF, symbol Device:C_Polarized
- added C19: 47µF, symbol Device:C
- added C21: 0.01µf, symbol Device:C
- added C4: 0.01 µF, symbol Device:C
- added C6: 0.01µF, symbol Device:C
- added IC1: MCP2517FDT-H_SL, SOIC127P600X175-14N, symbol CANFDControllerNew:MCP2517FDT-H_SL
- added R4, R7: 10k, symbol Device:R
- added R5, R6: ~62k, symbol Device:R
- added U10: MCP3204-CI/P, PDIP14_300MC_MCH, symbol ADC4Channel:MCP3204-CI_P
- added U6: DSC1001DL5-020.0000T, LV-Sensor-Footprints-Lib:CDFN4_2P5X2_MCH, symbol LV-Sensor-Lib:DSC1001DL5-020.0000T
- added U7: ADS114S06BIPBSR, LV-Sensor-Footprints-Lib:PBS0032A_N, symbol LV-Sensor-Lib:ADS114S06BIPBSR
- added U8: LM2662MX/NOPB, LV-Sensor-Footprints-Lib:M08A, symbol LV-Sensor-Lib:LM2662MX_NOPB
Connections:
- net +2V5: now also C17.2, U7.23 (REFOUT), U7.26 (AVDD), U8.1 (FC), U8.8 (V+)
- net +3.3V: now also C1.2, C2.2, C7.2, IC1.14 (VDD), U6.4 (VDD), U7.15 (IOVDD), U7.16 (DVDD), U7.18 (RESET_N)
- net +5V: now also U10.13 (VREF), U10.14 (VDD)
- net GND: now also U9.8 (STBY), C1.1, C18.2, C19.2, C2.1, C21.1, C4.1, C6.1, C7.1, IC1.7 (VSS), R4.2, R7.2, U10.12 (AGND), U6.2 (GND), U7.14 (DGND), U7.17 (CLK), U7.8 (START_SYNC), U8.3 (GND), U8.4 (C1-), U8.6 (LV)
- net at J16.1 (VBUS), U3.15 (VCC): now also C6.2
- net at U2.14 (PA18_/_A7): now also IC1.12 (SDO), U10.10 (DOUT), U7.12 (DOUT_DRDY_N)
- net at U2.13 (PA17_/_A9): now also IC1.10 (SCK), U10.11 (CLK), U7.11 (SCLK)
- net at U2.17 (PA22_/_A4): now also IC1.11 (SDI), U10.9 (DIN), U7.10 (DIN)
- net at U9.1 (TXD): now also IC1.1 (TXCAN)
- net at U9.4 (RXD): now also IC1.2 (RXCAN)
- net at R1.1, SW1.1, U2.4 (NRST): now also C4.2
- net at U2.8 (PA2): now also U7.9 (CS_N)
- net CAN_H: no longer names the net of U9.7 (CANH)
- net CAN_L: no longer names the net of U9.6 (CANL)
- net PA0: no longer names the net of U2.11 (PA0)
- net PA0: now also IC1.13 (NCS)
- net PA1: no longer names the net of U2.12 (PA1)
- net PA1: now also U10.8 (CS/SHDN)
- new net: C17.1, C19.1, U7.24 (REFCOM), U7.27 (AVSS), U8.5 (OUT)
- new net: IC1.6 (OSC1), U6.3 (OUT)
- new net: R6.2, R7.1, U7.6 (AIN1)
- new net: R4.1, R5.2, U7.7 (AIN0)
- new net: C18.1, U8.2 (C1+)
- new net: C21.2, U10.7 (DGND)
- no-connect marks 30 -> 16
Other:
- note added: "-2V5 OUT"
- note added: "2Inputs_[-18,18V] Ratio: 6.2"
- note added: "4Inputs_[0,5V]"
- note added: "A0_Input"
- note added: "A1_Input"
- note added: "CS FOR ADC4"
- note added: "SCK"
- note added: "SDI"
- note added: "SDO"
- note removed: "NEED TO PROTECT THE 12V INPUT"
- note removed: "pg.4 : leave floating?"
- moved on the sheet: C10, C11, C12, C13, C14, C15, C16, C20, C3, C5, C8, C9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

Commit message: rgwg
fixxes
Connections:
- net +3.3V is gone; now on net 3V3 OUT: C1.2, C2.2, C5.1, C7.2, C8.1, IC1.14 (VDD), R1.2, U2.9 (VDD), U6.4 (VDD), U7.15 (IOVDD), U7.16 (DVDD), U7.18 (RESET_N), U9.5 (VIO)
- net +5V is gone; now on net 5V out: U10.13 (VREF), U10.14 (VDD), U9.3 (VCC)
- net 2V5 OUT is gone; now on net +2V5: C20.1, U5.5 (OUT)
Other:
- note added: "2V5"
- note added: "3.3V"
- note added: "3.3V In"
- note added: "5V"
- moved on the sheet: C1, C10, C11, C12, C13, C14, C15, C16, C17, C18, C19, C2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

Commit message: fthft
thhf
Parts:
- added J1, J2, J3: Screw_Terminal_01x02, TerminalBlock_MetzConnect:TerminalBlock_MetzConnect_Type059_RT06302HBWC_1x02_P3.50mm_Horizontal, symbol Connector:Screw_Terminal_01x02
- added R10, R11, R12, R13, R14, R15, R8, R9: 0.5k, symbol Device:R
- added R16, R17: 1k, symbol Device:R
Connections:
- net GND: now also U8.7 (OSC)
- net at R6.2, R7.1: now also R17.2; no longer U7.6 (AIN1)
- net at U10.1 (CH0): now also R14.1
- net at U10.2 (CH1): now also R12.1
- net at U10.3 (CH2): now also R10.1
- net at U10.4 (CH3): now also R8.1
- net at R6.1: now also J2.2 (Pin_2)
- net at R5.1: now also R4.1, R16.2
- new net: J2.1 (Pin_1), R5.2
- new net: R8.2, R9.1
- new net: R10.2, R11.1
- new net: J3.2 (Pin_2), R11.2
- new net: R17.1, U7.6 (AIN1)
- new net: R16.1, U7.7 (AIN0)
- new net: R14.2, R15.1
- new net: J1.2 (Pin_2), R15.2
- new net: J1.1 (Pin_1), R13.2
- new net: J3.1 (Pin_1), R9.2
- new net: R12.2, R13.1
- no-connect marks 16 -> 31
Other:
- moved on the sheet: R4, R5, R6, R7

Commit message: sdfs
sfds
Parts:
- removed C19: 47µF, symbol Device:C
- removed C6: 0.01µF, symbol Device:C
- removed R11, R13, R15, R9: 0.5k, symbol Device:R
- removed R16, R17: 1k, symbol Device:R
- added C19: 47µF, ADC2_AND_4:A750_5X7_, symbol Device:C_Polarized
- added C22: 10uF, Capacitor_SMD:C_1206_3216Metric_Pad1.33x1.80mm_HandSolder, symbol Device:C_Small
- added C23: 100nF, Capacitor_SMD:C_1206_3216Metric_Pad1.33x1.80mm_HandSolder, symbol Device:C
- added C24, C25: 22uF, Capacitor_SMD:C_1206_3216Metric_Pad1.33x1.80mm_HandSolder, symbol Device:C
- added D1, D2, D3, D4, D5, D6, D7, D8: BAT54S, Package_TO_SOT_SMD:SOT-23, symbol Diode:BAT54S
- added J3, J5: Screw_Terminal_01x02, TerminalBlock_MetzConnect:TerminalBlock_MetzConnect_Type059_RT06302HBWC_1x02_P3.50mm_Horizontal, symbol Connector:Screw_Terminal_01x02
- added L1: 4.7uH, Inductor_SMD:L_TDK_NLV25_2.5x2.0mm, symbol Device:L
- added R20, R23: ~62k, Resistor_SMD:R_1206_3216Metric_Pad1.30x1.75mm_HandSolder, symbol Device:R
- added R21, R22: 10k, Resistor_SMD:R_1206_3216Metric_Pad1.30x1.75mm_HandSolder, symbol Device:R
- added R24: 10k, Resistor_SMD:R_2010_5025Metric_Pad1.40x2.65mm_HandSolder, symbol Device:R
- added U0: AP63205WU-7, LV-Sensor-Footprints-Lib:AP6320xWU-7_DIO, symbol LV-Sensor-Lib:AP63205WU-7
- C1, C2: footprint (none) -> ADC2_AND_4:CAPC3216X125N; mouser (none) -> https://www.mouser.com/ProductDetail/Murata-Electronics/GRT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
- C17: footprint (none) -> ADC2_AND_4:CAPC3216X100N; Mouser (none) -> https://www.mouser.com/ProductDetail/Samsung-Electro-Mechan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
- C18: footprint (none) -> ADC2_AND_4:A750_5X7_; mouser (none) -> https://www.mouser.com/ProductDetail/KEMET/A750BG227M0JAAE0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
- C21, C4: footprint (none) -> ADC2_AND_4:CAPC3216X140N; Field5 (none) -> https://www.mouser.com/ProductDetail/Samsung-Electro-Mechan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
- C7: footprint (none) -> ADC2_AND_4:CAPC3216X125N
- IC1: footprint SOIC127P600X175-14N -> ADC2_AND_4:CAN_FD_SOIC127P600X175-14N
- R10, R12, R14: value 0.5k -> 20k; footprint (none) -> Resistor_SMD:R_2010_5025Metric_Pad1.40x2.65mm_HandSolder
- R4: footprint (none) -> Resistor_SMD:R_1206_3216Metric_Pad1.30x1.75mm_HandSolder; mouser (none) -> https://www.mouser.com/ProductDetail/Vishay/CRCW120610K0FKE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
- R5: footprint (none) -> Resistor_SMD:R_1206_3216Metric_Pad1.30x1.75mm_HandSolder; mouser (none) -> https://www.mouser.com/ProductDetail/Bourns/CR1206-JW-623EL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
- R6, R7: footprint (none) -> Resistor_SMD:R_1206_3216Metric_Pad1.30x1.75mm_HandSolder
- R8: value 0.5k -> 20k; footprint (none) -> Resistor_SMD:R_2010_5025Metric_Pad1.40x2.65mm_HandSolder; mouser (none) -> https://www.mouser.com/ProductDetail/YAGEO/RC2010JK-071KL?q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
- SW1: footprint (none) -> Button_Switch_SMD:SW_SPST_PTS645Sx43SMTR92; mouser (none) -> https://www.mouser.com/ProductDetail/CK/KSC251J-SP-DELTA-LF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
- TP1, TP2: footprint (none) -> TestPoint:TestPoint_Pad_D2.0mm
- U10: footprint PDIP14_300MC_MCH -> ADC2_AND_4:PDIP14_300MC_MCH
- renumbered J3 to J2, J2 to J4, L1 to L3
Connections:
- net +12V: now also C22.1, U0.2 (EN), U0.3 (VIN)
- net +2V5: now also D1.2 (K), D2.2 (K), D3.2 (K), D4.2 (K)
- net GND: now also C19.2, C22.2, C24.1, C25.1, D5.1 (A), D6.1 (A), D7.1 (A), D8.1 (A), J5.2 (Pin_2), R21.2, R22.2, U0.4 (GND)
- net at R8.1, U10.4 (CH3): now also D5.3 (COM)
- net at R8.2: now also J2.1 (Pin_1)
- net -2V5: now reaches C17.1, U7.24 (REFCOM), U7.27 (AVSS), U8.5 (OUT)
- net -2V5: now also C19.1, D1.1 (A), D2.1 (A), D3.1 (A), D4.1 (A)
- net at R10.2: now also J2.2 (Pin_2)
- net at U7.4 (AIN3): now also D4.3 (COM), R22.1, R23.2
- net at U7.5 (AIN2): now also D3.3 (COM), R20.1, R21.1
- net at U7.6 (AIN1): now also R6.2, R7.1, D2.3 (COM)
- net at U7.7 (AIN0): now also R4.1, R5.1, D1.3 (COM)
- net at J16.1 (VBUS): no longer U3.15 (VCC)
- net at R14.2: now also J1.2 (Pin_2)
- net at R14.1, U10.1 (CH0): now also D8.3 (COM)
- net at R12.1, U10.2 (CH1): now also D7.3 (COM)
- net at R10.1, U10.3 (CH2): now also D6.3 (COM)
- net at J1.1 (Pin_1): now also R12.2
- net 3V3 OUT renamed +3V3
- net 5V out renamed +5V
- net +5V: now also C24.2, C25.2, D5.2 (K), D6.2 (K), D7.2 (K), D8.2 (K), J5.1 (Pin_1), L1.1, R24.1, U0.1 (FB)
- new net: R24.2, U3.15 (VCC)
- new net: J3.1 (Pin_1), R20.2
- new net: C23.2, L1.2, U0.5 (SW)
- new net: C23.1, U0.6 (BST)
- new net: J3.2 (Pin_2), R23.1
- no-connect marks 31 -> 33
Other:
- moved on the sheet: J1, J2, R8

Commit message: gfh
fghfg

Co-Authored-By: Manish Shrestha <manish.shr006@gmail.com>
Parts:
- removed C13, C3: 10uF, Capacitor_SMD:C_1206_3216Metric_Pad1.33x1.80mm_HandSolder, symbol Device:C_Small
- removed C14: 100nF, Capacitor_SMD:C_1206_3216Metric_Pad1.33x1.80mm_HandSolder, symbol Device:C
- removed C15: 22uF, Capacitor_SMD:C_1206_3216Metric_Pad1.33x1.80mm_HandSolder, symbol Device:C
- removed C16, C20: 1uF, Capacitor_SMD:C_1206_3216Metric_Pad1.33x1.80mm_HandSolder, symbol Device:C_Small
- removed L2, L3: 4.7uH, Inductor_SMD:L_TDK_NLV25_2.5x2.0mm, symbol Device:L
- removed U1: AP63205WU-7, LV-Sensor-Footprints-Lib:AP6320xWU-7_DIO, symbol LV-Sensor-Lib:AP63205WU-7
- removed U4: AP63203WU-7, LV-Sensor-Footprints-Lib:AP6320xWU-7_DIO, symbol LV-Sensor-Lib:AP63203WU-7
- removed U5: TLV77325PDBVR, LV-Sensor-Footprints-Lib:DBV0005A-IPC_A, symbol LV-Sensor-Lib:TLV77325PDBVR
- added C13: 1uF, Capacitor_SMD:C_1206_3216Metric_Pad1.33x1.80mm_HandSolder, symbol Device:C
- added C3, C6: 10uF, Capacitor_SMD:C_1206_3216Metric_Pad1.33x1.80mm_HandSolder, symbol Device:C
- added IC2: L78L05ABUTR, Package_TO_SOT_SMD:SOT-89-3_Handsoldering, symbol LV-Sensor-Lib:L78L05ABUTR
- added IC3: TLV74133PDBVR, Package_TO_SOT_SMD:SOT-23-5_HandSoldering, symbol LV-Sensor-Lib:TLV74133PDBVR
- added IC4: TLV74125PDBVR, Package_TO_SOT_SMD:SOT-23-5_HandSoldering, symbol LV-Sensor-Lib:TLV74125PDBVR
- added J6: Screw_Terminal_01x02, TerminalBlock_MetzConnect:TerminalBlock_MetzConnect_Type059_RT06302HBWC_1x02_P3.50mm_Horizontal, symbol Connector:Screw_Terminal_01x02
- added R9: 1k, Resistor_SMD:R_2010_5025Metric_Pad1.40x2.65mm_HandSolder, symbol Device:R
- C10: value 100nF -> 1uF; mouser https://www.mouser.com/ProductDetail/Murata-Electronics/GRT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 -> (none); specs 0.1 uF, 1% tolerance, -55 to +125C -> (none); unit x10 0.583 -> (none)
- C11: value 22uF -> 1uF; mouser https://www.mouser.com/ProductDetail/Samsung-Electro-Mechan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 -> (none); specs 22 uF, 25VDC, +/-10%, -55C to +85C -> (none); unit x10 0.076 -> (none)
- C12: value 22uF -> 1uF; Field5 (none) -> https://www.mouser.com/ProductDetail/KEMET/C1206C105K4RACTM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; mouser https://www.mouser.com/ProductDetail/Samsung-Electro-Mechan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 -> (none); specs 22 uF, 25VDC, +/-10%, -55C to +85C -> (none); unit x10 0.076 -> (none)
- C8, C9: footprint Capacitor_SMD:C_1206_3216Metric_Pad1.33x1.80mm_HandSolder -> ADC2_AND_4:CAPC3216X125N
- D1: footprint Package_TO_SOT_SMD:SOT-23 -> Package_TO_SOT_SMD:SOT-23-3; Field5 (none) -> https://www.mouser.com/ProductDetail/Diotec-Semiconductor/B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
- D2, D3, D4, D5, D6, D7, D8: footprint Package_TO_SOT_SMD:SOT-23 -> Package_TO_SOT_SMD:SOT-23-3
- R10, R12, R14: footprint Resistor_SMD:R_2010_5025Metric_Pad1.40x2.65mm_HandSolder -> Resistor_SMD:R_1206_3216Metric_Pad1.30x1.75mm_HandSolder
- R8: footprint Resistor_SMD:R_2010_5025Metric_Pad1.40x2.65mm_HandSolder -> Resistor_SMD:R_1206_3216Metric_Pad1.30x1.75mm_HandSolder; mouser https://www.mouser.com/ProductDetail/YAGEO/RC2010JK-071KL?q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 -> https://www.mouser.com/ProductDetail/Vishay/CRCW120620K0JNE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
Connections:
- net +12V: now also J6.1 (Pin_1), R9.1
- net +2V5: now also C13.1, IC4.5 (OUT)
- net +3V3: now also C11.1, C12.1, IC3.5 (OUT), IC4.1 (IN), IC4.3 (EN)
- net +5V: now also C10.2, C6.2, IC2.1 (VOUT), IC3.1 (IN), IC3.3 (EN); no longer C11.2, C12.2, C24.2, C25.2, J5.1 (Pin_1), L1.1, U0.1 (FB)
- net GND: now also C10.1, C11.2, C12.2, C13.2, C3.1, C6.1, IC2.2 (GND_1), IC2.4 (GND_2), IC3.2 (GND), IC4.2 (GND), J6.2 (Pin_2); no longer C11.1, C12.1
- new net: C3.2, IC2.3 (VIN), R9.2
- new net 5V out: C24.2, C25.2, J5.1 (Pin_1), L1.1, U0.1 (FB)
Other:
- note removed: "3V3 IN"

Commit message: dfggd
fd
Parts:
- removed J6: Screw_Terminal_01x02, TerminalBlock_MetzConnect:TerminalBlock_MetzConnect_Type059_RT06302HBWC_1x02_P3.50mm_Horizontal, symbol Connector:Screw_Terminal_01x02
- added J6: 43650-0415, ADC2_AND_4:43650-04YY_151617, symbol LV-Sensor-Lib:43650-0415
Connections:
- net +12V: now also J6.1
- net GND: now also J6.2
- net CAN_L: now reaches U9.6 (CANL)
- net CAN_L: now also J6.4
- net CAN_H: now reaches U9.7 (CANH)
- net CAN_H: now also J6.3

Commit message: fdg
dgf
Parts:
- removed J6: 43650-0415, ADC2_AND_4:43650-04YY_151617, symbol LV-Sensor-Lib:43650-0415
- added J6: 43650-0401, ADC2_AND_4:43650-04YY_151617, symbol LV-Sensor-Lib:43650-0401
Connections:
- net +12V: now also J6.1
- net CAN_H: now also J6.3
- net CAN_L: now also J6.4
- net GND: now also J6.2
Changed lines of the file:
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@@
 	(wire
 		(pts
-			(xy 76.2 53.34) (xy 81.28 53.34)
-		)
-		(stroke
-			(width 0)
-			(type default)
-		)
-	)
-	(wire
-		(pts
 			(xy 276.86 73.66) (xy 270.51 73.66)
 		)
@@
 	(wire
 		(pts
-			(xy 76.2 55.88) (xy 81.28 55.88)
-		)
-		(stroke
-			(width 0)
-			(type default)
-		)
-	)
-	(wire
-		(pts
 			(xy 402.59 134.62) (xy 405.13 134.62)
 		)
@@
 	(global_label "CAN_H"
 		(shape input)
-		(at 81.28 53.34 0)
+		(at 48.26 53.34 0)
 		(fields_autoplaced yes)
 		(effects
@@
 		)
 		(property "Intersheetrefs" "${INTERSHEET_REFS}"
-			(at 90.2524 53.34 0)
+			(at 57.2324 53.34 0)
 			(effects
 				(font
@@
 	(global_label "CAN_L"
 		(shape input)
-		(at 81.28 55.88 0)
+		(at 397.51 68.58 0)
 		(fields_autoplaced yes)
 		(effects
@@
 		)
 		(property "Intersheetrefs" "${INTERSHEET_REFS}"
-			(at 89.95 55.88 0)
+			(at 406.18 68.58 0)
 			(effects
 				(font
@@
 	(global_label "CAN_L"
 		(shape input)
-		(at 397.51 68.58 0)
+		(at 48.26 55.88 0)
 		(fields_autoplaced yes)
 		(effects
@@
 		)
 		(property "Intersheetrefs" "${INTERSHEET_REFS}"
-			(at 406.18 68.58 0)
+			(at 56.93 55.88 0)
 			(effects
 				(font
@@
 	)
 	(symbol
-		(lib_id "LV-Sensor-Lib:43650-0415")
-		(at 76.2 55.88 180)
-		(unit 1)
-		(exclude_from_sim no)
-		(in_bom yes)
-		(on_board yes)
-		(dnp no)
-		(fields_autoplaced yes)
-		(property "Reference" "J6"
-			(at 66.04 40.64 0)
-			(effects
-				(font
-					(size 1.27 1.27)
-				)
-			)
-		)
-		(property "Value" "43650-0415"
-			(at 66.04 43.18 0)
-			(effects
-				(font
-					(size 1.27 1.27)
-				)
-			)
-		)
-		(property "Footprint" "ADC2_AND_4:43650-04YY_151617"
-			(at 59.69 -39.04 0)
-			(effects
-				(font
-					(size 1.27 1.27)
-				)
-				(justify left top)
-				(hide yes)
-			)
-		)
-		(property "Datasheet" "https://www.molex.com/pdm_docs/sd/436500215_sd.pdf"
-			(at 59.69 -139.04 0)
-			(effects
-				(font
-					(size 1.27 1.27)
-				)
-				(justify left top)
-				(hide yes)
-			)
-		)
-		(property "Description" "Micro-Fit 3.0 Vertical Header, 3.00mm Pitch, Single Row, 4 Circuits, with PCB Polarizing Peg, Glow-Wire Capable, Black"
-			(at 76.2 55.88 0)
-			(effects
-				(font
-					(size 1.27 1.27)
-				)
-				(hide yes)
-			)
-		)
-		(property "Height" "9.9"
-			(at 59.69 -339.04 0)
-			(effects
-				(font
-					(size 1.27 1.27)
-				)
-				(justify left top)
-				(hide yes)
-			)
-		)
-		(property "Mouser Part Number" "538-43650-0415"
-			(at 59.69 -439.04 0)
-			(effects
-				(font
-					(size 1.27 1.27)
-				)
-				(justify left top)
-				(hide yes)
-			)
-		)
-		(property "Mouser Price/Stock" "https://www.mouser.co.uk/ProductDetail/Molex/43650-0415?qs=GEJyObWCoZgrB2DNhHHwDQ%3D%3D"
-			(at 59.69 -539.04 0)
-			(effects
-				(font
-					(size 1.27 1.27)
-				)
-				(justify left top)
-				(hide yes)
-			)
-		)
-		(property "Manufacturer_Name" "Molex"
-			(at 59.69 -639.04 0)
-			(effects
-				(font
-					(size 1.27 1.27)
-				)
-				(justify left top)
-				(hide yes)
-			)
-		)
-		(property "Manufacturer_Part_Number" "43650-0415"
-			(at 59.69 -739.04 0)
-			(effects
-				(font
-					(size 1.27 1.27)
-				)
-				(justify left top)
-				(hide yes)
-			)
-		)
-		(pin "3"
-		)
-		(pin "4"
-		)
-		(pin "2"
-		)
-		(pin "1"
-		)
-		(instances
-			(project ""
-				(path "/1afce36f-b357-4e2a-9166-a84df6dcc281"
-					(reference "J6")
-					(unit 1)
-				)
-			)
-		)
-	)
-	(symbol
 		(lib_id "Device:C_Small")
 		(at 182.88 59.69 0)
@@
 	(symbol
 		(lib_id "power:+12V")
-		(at 76.2 48.26 270)
+		(at 48.26 48.26 270)
 		(unit 1)
 		(exclude_from_sim no)
@@
 		(on_board yes)
 		(dnp no)
-		(fields_autoplaced yes)
 		(property "Reference" "#PWR051"
-			(at 72.39 48.26 0)
+			(at 44.45 48.26 0)
 			(effects
 				(font
@@
 		)
 		(property "Value" "+12V"
-			(at 80.01 48.2599 90)
+			(at 52.07 48.2599 90)
 			(effects
 				(font
@@
 		)
 		(property "Footprint" ""
-			(at 76.2 48.26 0)
+			(at 48.26 48.26 0)
 			(effects
 				(font
@@
 		)
 		(property "Datasheet" ""
-			(at 76.2 48.26 0)
+			(at 48.26 48.26 0)
 			(effects
 				(font
@@
 		)
 		(property "Description" "Power symbol creates a global label with name \"+12V\""
-			(at 76.2 48.26 0)
+			(at 48.26 48.26 0)
 			(effects
 				(font
@@
 		)
 		(instances
-			(project ""
+			(project "LV Sensor"
 				(path "/1afce36f-b357-4e2a-9166-a84df6dcc281"
 					(reference "#PWR051")
@@
 	(symbol
 		(lib_id "power:GND")
-		(at 76.2 50.8 90)
+		(at 48.26 50.8 90)
 		(unit 1)
 		(exclude_from_sim no)
@@
 		(fields_autoplaced yes)
 		(property "Reference" "#PWR052"
-			(at 82.55 50.8 0)
+			(at 54.61 50.8 0)
 			(effects
 				(font
@@
 		)
 		(property "Value" "GND"
-			(at 80.01 50.7999 90)
+			(at 52.07 50.7999 90)
 			(effects
 				(font
@@
 		)
 		(property "Footprint" ""
-			(at 76.2 50.8 0)
+			(at 48.26 50.8 0)
 			(effects
 				(font
@@
 		)
 		(property "Datasheet" ""
-			(at 76.2 50.8 0)
+			(at 48.26 50.8 0)
 			(effects
 				(font
@@
 		)
 		(property "Description" "Power symbol creates a global label with name \"GND\" , ground"
-			(at 76.2 50.8 0)
+			(at 48.26 50.8 0)
 			(effects
 				(font
@@
 		)
 		(instances
-			(project ""
+			(project "LV Sensor"
 				(path "/1afce36f-b357-4e2a-9166-a84df6dcc281"
 					(reference "#PWR052")
@@
 					(unit 1)
 				)
+			)
+		)
+	)
+	(symbol
+		(lib_id "LV-Sensor-Lib:43650-0401")
+		(at 48.26 55.88 180)
+		(unit 1)
+		(exclude_from_sim no)
+		(in_bom yes)
+		(on_board yes)
+		(dnp no)
+		(fields_autoplaced yes)
+		(property "Reference" "J6"
+			(at 38.1 40.64 0)
+			(effects
+				(font
+					(size 1.27 1.27)
+				)
+			)
+		)
+		(property "Value" "43650-0401"
+			(at 38.1 43.18 0)
+			(effects
+				(font
+					(size 1.27 1.27)
+				)
+			)
+		)
+		(property "Footprint" "ADC2_AND_4:43650-04YY_151617"
+			(at 31.75 -39.04 0)
+			(effects
+				(font
+					(size 1.27 1.27)
+				)
+				(justify left top)
+				(hide yes)
+			)
+		)
+		(property "Datasheet" "https://www.molex.com/pdm_docs/sd/436500200_sd.pdf"
+			(at 31.75 -139.04 0)
+			(effects
+				(font
+					(size 1.27 1.27)
+				)
+				(justify left top)
+				(hide yes)
+			)
+		)
+		(property "Description" "Micro-Fit 3.0 Right-Angle Header, 3.00mm Pitch, Single Row, 4 Circuits, with Snap-in Plastic Peg PCB Lock, Glow-Wire Capable, Black"
+			(at 48.26 55.88 0)
+			(effects
+				(font
+					(size 1.27 1.27)
+				)
+				(hide yes)
+			)
+		)
+		(property "Height" "5.57"
+			(at 31.75 -339.04 0)
+			(effects
+				(font
+					(size 1.27 1.27)
+				)
+				(justify left top)
+				(hide yes)
+			)
+		)
+		(property "Mouser Part Number" "538-43650-0401"
+			(at 31.75 -439.04 0)
+			(effects
+				(font
+					(size 1.27 1.27)
+				)
+				(justify left top)
+				(hide yes)
+			)
+		)
+		(property "Mouser Price/Stock" "https://www.mouser.co.uk/ProductDetail/Molex/43650-0401?qs=tCVB0Dok1YBvOr8VX%2FzPCg%3D%3D"
+			(at 31.75 -539.04 0)
+			(effects
+				(font
+					(size 1.27 1.27)
+				)
+				(justify left top)
+				(hide yes)
+			)
+		)
+		(property "Manufacturer_Name" "Molex"
+			(at 31.75 -639.04 0)
+			(effects
+				(font
+					(size 1.27 1.27)
+				)
+				(justify left top)
+				(hide yes)
+			)
+		)
+		(property "Manufacturer_Part_Number" "43650-0401"
+			(at 31.75 -739.04 0)
+			(effects
+				(font
+					(size 1.27 1.27)
+				)
+				(justify left top)
+				(hide yes)
+			)
+		)
+		(pin "4"
+		)
+		(pin "1"
+		)
+		(pin "3"
+		)
+		(pin "2"
+		)
+		(instances
+			(project ""
+				(path "/1afce36f-b357-4e2a-9166-a84df6dcc281"
+					(reference "J6")
+					(unit 1)
+				)
