File: kicad/LV Sensor.kicad_pcb (KiCad board)
At the start: 2 copper layers, 42 parts, among them U1 AP63205WU-7, U10 LM2662MX/NOPB, U2 XMSM0C1104SPW20R, U3 FT231XS-R, U4 AP63203WU-7, U5 TLV77325PDBVR, U6 MCP2518FD-xJHA, U7 DSC1001DL5-020.0000T, U8 ADS114S06BIPBSR, U9 ATA6561-GAQW-N

Commit message: trh
thrsth
Parts:
- moved R1 69.0 mm to (114.0, 30.8), turned to 180 degrees
- moved U6 65.6 mm to (109.4, 38.0)
- moved R3 64.7 mm to (147.4, 41.1), turned to 180 degrees
- moved C1 64.6 mm to (158.8, 100.1)
- moved U2 63.0 mm to (118.6, 37.2)
- moved R2 58.8 mm to (147.4, 43.9)
- moved U9 55.5 mm to (99.9, 36.3)
- moved U8 54.8 mm to (118.2, 48.0), turned to 135 degrees
- moved U10 48.9 mm to (77.4, 81.7)
- moved U3 45.6 mm to (155.5, 43.1), turned to 180 degrees
- moved U4 24.8 mm to (156.8, 75.8), turned to -90 degrees
- moved U1 20.1 mm to (151.8, 69.6), turned to -135 degrees
Routing:
- net GND: track 205.0 -> 0.00 mm
- net +3.3V: track 102.9 -> 0.00 mm, vias 4 -> 0
- net /3V3 OUT: track 77.9 -> 0.00 mm, vias 6 -> 0
- net Net-(U2-PA2): track 75.8 -> 0.00 mm, vias 2 -> 0
- net Net-(C1-Pad1): track 71.3 -> 0.00 mm, vias 2 -> 0
- net +5V: track 70.6 -> 0.00 mm, vias 4 -> 0
- net Net-(U1-SW): track 64.3 -> 0.00 mm, vias 3 -> 0
- net +12V: track 62.8 -> 0.00 mm
- net Net-(U2-NRST): track 60.9 -> 0.00 mm, vias 2 -> 0
- net /5V out: track 59.6 -> 0.00 mm, vias 3 -> 0
- net Net-(C4-Pad1): track 55.0 -> 0.00 mm, vias 2 -> 0
- net Net-(U4-SW): track 53.8 -> 0.00 mm, vias 3 -> 0
- net Net-(U4-BST): track 47.2 -> 0.00 mm, vias 4 -> 0
- net Net-(U10-C1-): track 44.9 -> 0.00 mm, vias 4 -> 0
- net Net-(U10-C1+): track 42.2 -> 0.00 mm, vias 2 -> 0
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
Commit message: 5y5y
45y45

Co-Authored-By: Manish Shrestha <manish.shr006@gmail.com>
Parts:
- U2: value XMSM0C1104SPW20R -> MCU
- moved U9 79.8 mm to (168.0, 78.0)
- moved U10 77.8 mm to (155.2, 78.0)
- moved R1 77.4 mm to (154.8, 96.5)
- moved U2 76.4 mm to (167.8, 95.6)
- moved U6 75.8 mm to (167.8, 86.3)
- moved U8 67.6 mm to (178.0, 79.6), turned to 0 degrees
- moved C5 61.4 mm to (160.4, 96.5)
- moved R3 60.4 mm to (184.9, 88.5), turned to 0 degrees
- moved U7 59.8 mm to (175.1, 85.9)
- moved C8 57.8 mm to (160.5, 92.5)
- moved C2 57.2 mm to (154.8, 92.5)
- moved U5 54.3 mm to (160.8, 87.6)
- moved U3 53.8 mm to (177.8, 92.0), turned to 90 degrees
- moved R2 53.3 mm to (180.2, 85.8)
- moved L2 34.4 mm to (99.9, 71.5), turned to 180 degrees
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
Commit message: sdfs
sfds
Parts:
- removed C26, C6: 100nF, Capacitor_SMD:C_1206_3216Metric_Pad1.33x1.80mm_HandSolder
- removed C27: 47uF, Capacitor_SMD:C_1206_3216Metric_Pad1.33x1.80mm_HandSolder
- added D1: BAT54S, Package_TO_SOT_SMD:SOT-23, F.Cu at (205.2, 85.0)
- added D2: BAT54S, Package_TO_SOT_SMD:SOT-23, F.Cu at (208.3, 81.9)
- added D3: BAT54S, Package_TO_SOT_SMD:SOT-23, F.Cu at (205.0, 78.1)
- added D4: BAT54S, Package_TO_SOT_SMD:SOT-23, F.Cu at (208.0, 74.7)
- added D5: BAT54S, Package_TO_SOT_SMD:SOT-23, F.Cu at (212.4, 71.4)
- added D6: BAT54S, Package_TO_SOT_SMD:SOT-23, F.Cu at (209.3, 66.4)
- added D7: BAT54S, Package_TO_SOT_SMD:SOT-23, F.Cu at (212.3, 61.4)
- added D8: BAT54S, Package_TO_SOT_SMD:SOT-23, F.Cu at (209.2, 56.6)
- added IC1: MCP2517FDT-H_SL, ADC2_AND_4:CAN_FD_SOIC127P600X175-14N, F.Cu at (191.4, 64.8)
- added J1: Screw_Terminal_01x02, TerminalBlock_MetzConnect:TerminalBlock_MetzConnect_Type059_RT06302HBWC_1x02_P3.50mm_Horizontal, F.Cu at (225.2, 60.6)
- added J16: USB_B_Micro, Connector_USB:USB_Micro-B_Amphenol_10118194-0001LF_Horizontal, F.Cu at (187.5, 91.2)
- added J2: Screw_Terminal_01x02, TerminalBlock_MetzConnect:TerminalBlock_MetzConnect_Type059_RT06302HBWC_1x02_P3.50mm_Horizontal, F.Cu at (225.1, 69.0)
- added J3: Screw_Terminal_01x02, TerminalBlock_MetzConnect:TerminalBlock_MetzConnect_Type059_RT06302HBWC_1x02_P3.50mm_Horizontal, F.Cu at (224.9, 77.3)
- added J4: Screw_Terminal_01x02, TerminalBlock_MetzConnect:TerminalBlock_MetzConnect_Type059_RT06302HBWC_1x02_P3.50mm_Horizontal, F.Cu at (224.8, 85.8)
- added J5: Screw_Terminal_01x02, TerminalBlock_MetzConnect:TerminalBlock_MetzConnect_Type059_RT06302HBWC_1x02_P3.50mm_Horizontal, F.Cu at (224.9, 93.9)
- added L1: 4.7uH, Inductor_SMD:L_TDK_NLV25_2.5x2.0mm, F.Cu at (123.5, 50.2)
- added R10: 20k, Resistor_SMD:R_2010_5025Metric_Pad1.40x2.65mm_HandSolder, F.Cu at (218.0, 65.8)
- added R12: 20k, Resistor_SMD:R_2010_5025Metric_Pad1.40x2.65mm_HandSolder, F.Cu at (218.1, 61.2)
- added R14: 20k, Resistor_SMD:R_2010_5025Metric_Pad1.40x2.65mm_HandSolder, F.Cu at (218.1, 56.5)
- added R20: ~62k, Resistor_SMD:R_1206_3216Metric_Pad1.30x1.75mm_HandSolder, F.Cu at (218.4, 78.3)
- added R21: 10k, Resistor_SMD:R_1206_3216Metric_Pad1.30x1.75mm_HandSolder, F.Cu at (213.2, 78.3)
- added R22: 10k, Resistor_SMD:R_1206_3216Metric_Pad1.30x1.75mm_HandSolder, F.Cu at (213.3, 74.6)
- added R23: ~62k, Resistor_SMD:R_1206_3216Metric_Pad1.30x1.75mm_HandSolder, F.Cu at (218.6, 74.6)
- added R24: 10k, Resistor_SMD:R_2010_5025Metric_Pad1.40x2.65mm_HandSolder, F.Cu at (146.1, 59.2)
- added R4: 10k, Resistor_SMD:R_1206_3216Metric_Pad1.30x1.75mm_HandSolder, F.Cu at (213.1, 85.7)
- added R5: ~62k, Resistor_SMD:R_1206_3216Metric_Pad1.30x1.75mm_HandSolder, F.Cu at (218.4, 85.7)
- added R6: ~62k, Resistor_SMD:R_1206_3216Metric_Pad1.30x1.75mm_HandSolder, F.Cu at (218.4, 82.0)
- added R7: 10k, Resistor_SMD:R_1206_3216Metric_Pad1.30x1.75mm_HandSolder, F.Cu at (213.1, 82.0)
- added R8: 20k, Resistor_SMD:R_2010_5025Metric_Pad1.40x2.65mm_HandSolder, F.Cu at (218.1, 70.4)
- added SW1: SW_Push, Button_Switch_SMD:SW_SPST_PTS645Sx43SMTR92, F.Cu at (186.5, 81.8)
- added TP1: TestPoint, TestPoint:TestPoint_Pad_D2.0mm, F.Cu at (192.1, 75.1)
- added TP2: TestPoint, TestPoint:TestPoint_Pad_D2.0mm, F.Cu at (192.0, 71.7)
- added U0: AP63205WU-7, LV-Sensor-Footprints-Lib:AP6320xWU-7_DIO, F.Cu at (115.0, 49.3)
- C1: value 47pF -> 0.1µF; footprint Capacitor_SMD:C_1206_3216Metric_Pad1.33x1.80mm_HandSolder -> ADC2_AND_4:CAPC3216X125N
- C17: value 1uF -> 330nF; footprint Capacitor_SMD:C_1206_3216Metric_Pad1.33x1.80mm_HandSolder -> ADC2_AND_4:CAPC3216X100N
- C18: value 0.1uF -> 47µF; footprint Capacitor_SMD:C_1206_3216Metric_Pad1.33x1.80mm_HandSolder -> ADC2_AND_4:A750_5X7_
- C19: value 15pF -> 47µF; footprint Capacitor_SMD:C_1206_3216Metric_Pad1.33x1.80mm_HandSolder -> ADC2_AND_4:A750_5X7_
- C2: value 100n -> 0.1µF; footprint Capacitor_SMD:C_1206_3216Metric_Pad1.33x1.80mm_HandSolder -> ADC2_AND_4:CAPC3216X125N
- C21: value 330nF -> 0.01µf; footprint Capacitor_SMD:C_1206_3216Metric_Pad1.33x1.80mm_HandSolder -> ADC2_AND_4:CAPC3216X140N
- C22: value 47uF -> 10uF
- C24, C25: value 100nF -> 22uF
- C4: value 47pF -> 0.01 µF; footprint Capacitor_SMD:C_1206_3216Metric_Pad1.33x1.80mm_HandSolder -> ADC2_AND_4:CAPC3216X140N
- C7: value 4.7uF -> 0.1µF; footprint Capacitor_SMD:C_1206_3216Metric_Pad1.33x1.80mm_HandSolder -> ADC2_AND_4:CAPC3216X125N
- U10: value LM2662MX/NOPB -> MCP3204-CI/P; footprint LV-Sensor-Footprints-Lib:M08A -> ADC2_AND_4:PDIP14_300MC_MCH
- U2: value MCU -> XMSM0C1104SPW20R
- U6: value MCP2518FD-xJHA -> DSC1001DL5-020.0000T; footprint LV-Sensor-Footprints-Lib:MCP2518FDT -> LV-Sensor-Footprints-Lib:CDFN4_2P5X2_MCH
- U7: value DSC1001DL5-020.0000T -> ADS114S06BIPBSR; footprint LV-Sensor-Footprints-Lib:CDFN4_2P5X2_MCH -> LV-Sensor-Footprints-Lib:PBS0032A_N
- U8: value ADS114S06BIPBSR -> LM2662MX/NOPB; footprint LV-Sensor-Footprints-Lib:PBS0032A_N -> LV-Sensor-Footprints-Lib:M08A
- moved C19 106.0 mm to (211.9, 91.4), turned to 0 degrees
- moved C18 99.7 mm to (205.8, 91.3)
- moved C17 94.3 mm to (200.4, 94.1), turned to 0 degrees
- moved U10 47.8 mm to (197.6, 56.1)
- moved C2 40.8 mm to (178.0, 58.9)
- moved C1 40.4 mm to (178.0, 55.7)
- moved R1 39.0 mm to (151.7, 57.7)
- moved U6 38.6 mm to (192.2, 56.4)
- moved C5 37.8 mm to (184.1, 67.0), turned to 180 degrees
- moved C4 37.7 mm to (155.7, 85.3), turned to 0 degrees
- moved R3 37.7 mm to (148.2, 80.0), turned to 90 degrees
- moved C7 37.3 mm to (151.4, 61.6), turned to 0 degrees
- moved C8 37.0 mm to (184.1, 63.9), turned to 180 degrees
- moved C22 35.4 mm to (99.0, 63.3), turned to 0 degrees
- moved U3 31.5 mm to (152.8, 73.0)
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- renumbered L1 to L3
Connections:
- C1 pad 1: Net-(C1-Pad1) -> GND
- C1 pad 2: GND -> +3V3
- C11 pad 2: /5V out -> +5V
- C12 pad 2: /5V out -> +5V
- C15 pad 2: /3V3 OUT -> +3V3
- C16 pad 1: /3V3 OUT -> +3V3
- C17 pad 1: Net-(U8-REFOUT) -> -2V5
- C17 pad 2: -2V5 -> +2V5
- C18 pad 1: GND -> Net-(U8-C1+)
- C18 pad 2: +3.3V -> GND
- C19 pad 1: +3V3 -> -2V5
- C2 pad 1: Net-(U2-NRST) -> GND
- C2 pad 2: GND -> +3V3
- C20 pad 1: /2V5 OUT -> +2V5
- C21 pad 1: +2V5 -> GND
- C21 pad 2: -2V5 -> Net-(U10-DGND)
- C22 pad 1: Net-(U10-C1+) -> +12V
- C22 pad 2: Net-(U10-C1-) -> GND
- C23 pad 1: +5V -> Net-(U0-BST)
- C23 pad 2: GND -> Net-(U0-SW)
- C24 pad 1: +3.3V -> GND
- C24 pad 2: GND -> +5V
- C25 pad 1: +5V -> GND
- C25 pad 2: GND -> +5V
- C4 pad 1: Net-(C4-Pad1) -> GND
- C4 pad 2: GND -> Net-(U2-NRST)
- C5 pad 1: +3.3V -> +3V3
- C7 pad 1: +5V -> GND
- C7 pad 2: GND -> +3V3
- C8 pad 1: +3.3V -> +3V3
- L2 pad 1: /3V3 OUT -> +3V3
- L3 pad 1: /5V out -> +5V
- R1 pad 2: +3.3V -> +3V3
- R2 pad 1: Net-(C4-Pad1) -> Net-(J16-D-)
- R3 pad 1: Net-(C1-Pad1) -> Net-(J16-D+)
- U1 pad 1: /5V out -> +5V
- U10 pad 1: +2V5 -> Net-(D8-COM)
- U10 pad 2: Net-(U10-C1+) -> Net-(D7-COM)
- U10 pad 3: GND -> Net-(D6-COM)
- U10 pad 4: Net-(U10-C1-) -> Net-(D5-COM)
- U10 pad 5: /-2V5 OUT -> unconnected-(U10-NC-Pad5)
- U10 pad 6: GND -> unconnected-(U10-NC-Pad6)
- U10 pad 7: unconnected-(U10-OSC-Pad7) -> Net-(U10-DGND)
- U10 pad 8: +2V5 -> Net-(U10-CS/SHDN)
- U2 pad 11: /PA0 -> Net-(IC1-NCS)
- U2 pad 12: /PA1 -> Net-(U10-CS/SHDN)
- U2 pad 13: Net-(U2-PA17_/_A9) -> Net-(IC1-SCK)
- U2 pad 14: Net-(U2-PA18_/_A7) -> Net-(IC1-SDO)
- U2 pad 17: Net-(U2-PA22_/_A4) -> Net-(IC1-SDI)
- U2 pad 9: +3.3V -> +3V3
- U3 pad 15: +5V -> Net-(U3-VCC)
- U4 pad 1: /3V3 OUT -> +3V3
- U5 pad 1: /3V3 OUT -> +3V3
- U5 pad 3: /3V3 OUT -> +3V3
- U5 pad 5: /2V5 OUT -> +2V5
- U6 pad 1: Net-(U6-TXCAN) -> unconnected-(U6-*STANDBY-Pad1)
- U6 pad 2: Net-(U6-RXCAN) -> GND
- U6 pad 4: Net-(U6-~{INT}) -> +3V3
- U7 pad 2: GND -> unconnected-(U7-AIN5-Pad2)
- U7 pad 3: Net-(U6-OSC1) -> unconnected-(U7-AIN4-Pad3)
- U7 pad 4: +3V3 -> Net-(D4-COM)
- U8 pad 1: unconnected-(U8-AINCOM-Pad1) -> +2V5
- U8 pad 2: unconnected-(U8-AIN5-Pad2) -> Net-(U8-C1+)
- U8 pad 3: unconnected-(U8-AIN4-Pad3) -> GND
- U8 pad 4: unconnected-(U8-AIN3-Pad4) -> GND
- U8 pad 5: unconnected-(U8-AIN2-Pad5) -> -2V5
- U8 pad 6: unconnected-(U8-AIN1-Pad6) -> GND
- U8 pad 7: unconnected-(U8-AIN0-Pad7) -> GND
- U8 pad 8: GND -> +2V5
- U9 pad 1: Net-(U6-TXCAN) -> Net-(IC1-TXCAN)
- U9 pad 4: Net-(U6-RXCAN) -> Net-(IC1-RXCAN)
- U9 pad 5: +3.3V -> +3V3
- U9 pad 6: /CAN_L -> unconnected-(U9-CANL-Pad6)
- U9 pad 7: /CAN_H -> unconnected-(U9-CANH-Pad7)
- U9 pad 8: Net-(U9-STBY) -> GND

Commit message: gfh
fghfg

Co-Authored-By: Manish Shrestha <manish.shr006@gmail.com>
Parts:
- removed C14: 100nF, Capacitor_SMD:C_1206_3216Metric_Pad1.33x1.80mm_HandSolder
- removed C15: 22uF, Capacitor_SMD:C_1206_3216Metric_Pad1.33x1.80mm_HandSolder
- removed C16, C20: 1uF, Capacitor_SMD:C_1206_3216Metric_Pad1.33x1.80mm_HandSolder
- removed L2, L3: 4.7uH, Inductor_SMD:L_TDK_NLV25_2.5x2.0mm
- removed U1: AP63205WU-7, LV-Sensor-Footprints-Lib:AP6320xWU-7_DIO
- removed U4: AP63203WU-7, LV-Sensor-Footprints-Lib:AP6320xWU-7_DIO
- removed U5: TLV77325PDBVR, LV-Sensor-Footprints-Lib:DBV0005A-IPC_A
- added C6: 10uF, Capacitor_SMD:C_1206_3216Metric_Pad1.33x1.80mm_HandSolder, F.Cu at (142.4, 96.4)
- added IC2: L78L05ABUTR, Package_TO_SOT_SMD:SOT-89-3_Handsoldering, F.Cu at (175.5, 45.8)
- added IC3: TLV74133PDBVR, Package_TO_SOT_SMD:SOT-23-5_HandSoldering, F.Cu at (161.9, 45.8)
- added IC4: TLV74125PDBVR, Package_TO_SOT_SMD:SOT-23-5_HandSoldering, F.Cu at (161.9, 50.5)
- added J6: Screw_Terminal_01x02, TerminalBlock_MetzConnect:TerminalBlock_MetzConnect_Type059_RT06302HBWC_1x02_P3.50mm_Horizontal, F.Cu at (134.4, 89.7)
- added R9: 1k, Resistor_SMD:R_2010_5025Metric_Pad1.40x2.65mm_HandSolder, F.Cu at (135.5, 96.8)
- C10: value 100nF -> 1uF
- C11, C12: value 22uF -> 1uF
- C13: value 10uF -> 1uF
- C8, C9: footprint Capacitor_SMD:C_1206_3216Metric_Pad1.33x1.80mm_HandSolder -> ADC2_AND_4:CAPC3216X125N
- D1, D2, D3, D4, D5, D6, D7, D8: footprint Package_TO_SOT_SMD:SOT-23 -> Package_TO_SOT_SMD:SOT-23-3
- R10, R12, R14, R8: footprint Resistor_SMD:R_2010_5025Metric_Pad1.40x2.65mm_HandSolder -> Resistor_SMD:R_1206_3216Metric_Pad1.30x1.75mm_HandSolder
Connections:
- C10 pad 1: Net-(U1-BST) -> GND
- C10 pad 2: Net-(U1-SW) -> +5V
- C11 pad 1: GND -> +3V3
- C11 pad 2: +5V -> GND
- C12 pad 1: GND -> +3V3
- C12 pad 2: +5V -> GND
- C13 pad 1: +12V -> +2V5
- C24 pad 2: +5V -> /5V out
- C25 pad 2: +5V -> /5V out
- C3 pad 1: +12V -> GND
- C3 pad 2: GND -> Net-(IC2-VIN)
- J5 pad 1: +5V -> /5V out
- L1 pad 1: +5V -> /5V out
- U0 pad 1: +5V -> /5V out

Commit message: gtugt
ugttu
Parts:
- moved IC2 105.0 mm to (70.8, 54.1), turned to 180 degrees
- moved C9 90.1 mm to (172.6, 94.2), turned to 0 degrees
- moved IC3 78.0 mm to (84.4, 54.2), turned to 180 degrees
- moved IC4 77.5 mm to (84.4, 49.4), turned to 180 degrees
- moved R1 29.7 mm to (175.8, 75.0), turned to -90 degrees
- moved U3 29.0 mm to (177.2, 88.6)
- moved C4 24.2 mm to (179.4, 80.6), turned to 90 degrees
- moved R24 12.8 mm to (133.7, 62.2)
- moved C7 12.8 mm to (139.0, 64.6)
- moved C5 9.28 mm to (179.4, 75.0), turned to 90 degrees
- moved C8 7.39 mm to (179.4, 69.6), turned to 90 degrees
- moved IC1 0.89 mm to (191.8, 64.0)
- moved TP2 0.40 mm to (192.4, 71.7)
- moved TP1 0.10 mm to (192.2, 75.1)

Commit message: dfggd
fd
Parts:
- J6: value Screw_Terminal_01x02 -> 43650-0415; footprint TerminalBlock_MetzConnect:TerminalBlock_MetzConnect_Type059_RT06302HBWC_1x02_P3.50mm_Horizontal -> ADC2_AND_4:43650-04YY_151617
- moved C10 91.5 mm to (170.0, 75.0), turned to 90 degrees
- moved IC2 91.0 mm to (157.3, 82.4)
- moved C12 88.3 mm to (165.3, 64.9), turned to 0 degrees
- moved C21 85.7 mm to (194.6, 59.9), turned to -90 degrees
- moved C11 85.6 mm to (164.8, 74.7), turned to 0 degrees
- moved IC3 84.9 mm to (165.6, 79.1)
- moved IC4 83.2 mm to (165.1, 69.5), turned to -90 degrees
- moved C13 80.9 mm to (160.4, 69.6), turned to 90 degrees
- moved C22 79.0 mm to (178.0, 61.2)
- moved C3 77.0 mm to (164.2, 85.8), turned to 90 degrees
- moved J5 73.5 mm to (159.8, 59.8), turned to 180 degrees
- moved C24 72.7 mm to (171.5, 64.9), turned to 180 degrees
- moved C25 72.6 mm to (171.5, 68.8), turned to 180 degrees
- moved C23 72.6 mm to (171.4, 61.2), turned to 180 degrees
- moved C7 62.0 mm to (199.6, 77.9), turned to 180 degrees
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Connections:
- U9 pad 6: unconnected-(U9-CANL-Pad6) -> CAN_L
- U9 pad 7: unconnected-(U9-CANH-Pad7) -> CAN_H

Commit message: fdg
dgf
Parts:
- J6: value 43650-0415 -> 43650-0401
- moved L1 13.2 mm to (176.6, 66.3)
- moved J6 8.72 mm to (153.3, 66.6), turned to -90 degrees
- moved J5 6.58 mm to (166.3, 58.8)
- moved U0 6.51 mm to (176.4, 61.8)
- moved C22 3.40 mm to (181.3, 61.8)
Routing:
- net Net-(D3-COM): track 0.00 -> 62.1 mm
- net GND: track 0.00 -> 49.6 mm
- net -2V5: track 0.00 -> 34.4 mm
- net Net-(D2-COM): track 0.00 -> 25.9 mm, vias 0 -> 1
- net Net-(D4-COM): track 0.00 -> 25.6 mm
- net Net-(D1-COM): track 0.00 -> 20.0 mm, vias 0 -> 1
- net Net-(J4-Pin_2): track 0.00 -> 12.8 mm
- net Net-(J3-Pin_2): track 0.00 -> 11.3 mm
- net Net-(J4-Pin_1): track 0.07 -> 9.59 mm
- net Net-(J3-Pin_1): track 0.00 -> 8.49 mm
- net +2V5: track 0.00 -> 8.44 mm
- net Net-(D6-COM): track 0.00 -> 6.26 mm
- net Net-(D8-COM): track 0.00 -> 6.25 mm
- net Net-(J2-Pin_1): track 0.00 -> 6.11 mm
- net Net-(J1-Pin_2): track 0.00 -> 5.80 mm
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
Commit message: finalized changes
Parts:
- removed U2: XMSM0C1104SPW20R, LV-Sensor-Footprints-Lib:TSSOP20_PW_TEX
- added IC5: MSPM0C1104SDGS20R, LV-Sensor-Footprints-Lib:SOP50P490X110-20N, F.Cu at (184.2, 75.8)
- J6: footprint ADC2_AND_4:43650-04YY_151617 -> LV-Sensor-Footprints-Lib:43650-04_00,01,02_
- TP1, TP2: moved to B.Cu
- moved C22 30.6 mm to (151.3, 67.7), turned to -90 degrees
- moved L1 25.8 mm to (153.4, 77.8), turned to 0 degrees
- moved C3 22.3 mm to (160.4, 63.9), turned to 0 degrees
- moved U0 22.2 mm to (155.1, 67.7), turned to -90 degrees
- moved C25 22.2 mm to (153.6, 81.9)
- moved C24 21.3 mm to (151.9, 73.2), turned to -90 degrees
- moved C13 21.0 mm to (161.6, 90.6), turned to 180 degrees
- moved C23 20.2 mm to (155.2, 73.2), turned to -90 degrees
- moved C6 19.6 mm to (161.0, 72.1), turned to 0 degrees
- moved R22 19.4 mm to (212.8, 94.0), turned to 90 degrees
- moved D4 19.3 mm to (208.1, 94.0), turned to -90 degrees
- moved R23 19.2 mm to (217.9, 93.8), turned to 180 degrees
- moved C12 18.6 mm to (165.2, 83.5), turned to 90 degrees
- moved C1 18.0 mm to (195.7, 58.3), turned to -90 degrees
- moved C18 17.7 mm to (188.3, 94.2)
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Connections:
- C18 pad 2: GND -> Net-(U8-C1-)
- IC1 pad 13: Net-(IC1-NCS) -> CS_CAN
- R20 pad 2: Net-(J3-Pin_1) -> Net-(J3-Pin_2)
- R23 pad 1: Net-(J3-Pin_2) -> Net-(J3-Pin_1)
- R5 pad 2: Net-(J4-Pin_1) -> Net-(J4-Pin_2)
- R6 pad 1: Net-(J4-Pin_2) -> Net-(J4-Pin_1)
- U10 pad 8: Net-(U10-CS/SHDN) -> CS_ADC4
- U3 pad 2: /UART0_RTS -> UART0_RTS
- U3 pad 20: /UART0_TX -> UART0_TX
- U3 pad 4: /UART0_RX -> UART0_RX
- U3 pad 9: /UART0_CTS -> UART0_CTS
- U7 pad 9: Net-(U2-PA2) -> CS_ADC8
- U8 pad 4: GND -> Net-(U8-C1-)
Routing:
- net +5V: track 0.00 -> 127.5 mm
- net +3V3: track 0.00 -> 116.3 mm
- net +2V5: track 8.44 -> 84.3 mm, vias 0 -> 4
- net Net-(IC1-SDI): track 0.00 -> 56.9 mm, vias 0 -> 1
- net GND: track 49.6 -> 0.00 mm
- net Net-(IC1-SDO): track 0.00 -> 43.7 mm, vias 0 -> 1
- net Net-(D3-COM): track 62.1 -> 22.0 mm
- net Net-(IC1-SCK): track 0.00 -> 38.6 mm, vias 0 -> 1
- net CS_CAN: track 0.00 -> 38.6 mm, vias 0 -> 2
- net /5V out: track 0.00 -> 36.6 mm
- net Net-(D5-COM): track 3.43 -> 31.3 mm
- net Net-(IC2-VIN): track 0.00 -> 27.6 mm
- net CS_ADC4: track 0.00 -> 27.4 mm, vias 0 -> 1
- net UART0_CTS: track 0.00 -> 24.0 mm, vias 0 -> 2
- net +12V: track 0.00 -> 22.5 mm
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Other:
- board outline added: 80.3 x 45.9 mm
